File: PCB/ROwen_Power.brd (EAGLE design)
At the start: 100 x 80 mm, 41 parts, among them CON1 MLW14_90°, CON10 WAGO256, CON11 WAGO256, CON12 WAGO256, CON2 WAGO256, CON3 WAGO256, CON4 WAGO256, CON5 WAGO256, CON6 WAGO256, CON7 WAGO256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

Commit message: Polygon improvement
Parts:
- R10: value 330 -> 360
- R12, R7, R8, R9: value 180 -> 220
Changed lines of the file:
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@@
 <element name="R5" library="resistor" package="0207/10" value="330" x="27.94" y="62.23" rot="R225"/>
 <element name="R6" library="resistor" package="0207/10" value="330" x="27.94" y="50.8" rot="R225"/>
-<element name="R7" library="resistor" package="0207/10" value="180" x="74.93" y="71.12" rot="R270"/>
-<element name="R8" library="resistor" package="0207/10" value="180" x="78.105" y="59.69" rot="R180"/>
-<element name="R9" library="resistor" package="0207/10" value="180" x="78.105" y="48.26" rot="R180"/>
+<element name="R7" library="resistor" package="0207/10" value="220" x="74.93" y="71.12" rot="R270"/>
+<element name="R8" library="resistor" package="0207/10" value="220" x="78.105" y="59.69" rot="R180"/>
+<element name="R9" library="resistor" package="0207/10" value="220" x="78.105" y="48.26" rot="R180"/>
 <element name="T1" library="kumen" package="TO220" value="BTA16" x="38.1" y="62.23" rot="R90"/>
 <element name="T2" library="kumen" package="TO220" value="BTA16" x="38.1" y="50.8" rot="R90"/>
@@
 <element name="TR1" library="#PaJa_30" package="TRHEI304" value="TRHEI304-1" x="69.85" y="17.78" rot="R90"/>
 <element name="CON1" library="#PaJa_konektory" package="MLW14A" value="MLW14_90°" x="92.71" y="54.61" rot="R270"/>
-<element name="R10" library="resistor" package="0207/10" value="330" x="53.34" y="36.83" rot="R180"/>
+<element name="R10" library="resistor" package="0207/10" value="360" x="53.34" y="36.83" rot="R180"/>
 <element name="OK4" library="optocoupler" package="DIL06" value="MOC3041M" x="66.04" y="39.37" rot="R90">
 <attribute name="OC_NEWARK" value="78K6090" x="69.85" y="27.94" size="1.778" layer="27" rot="R90" display="off"/>
@@
 <element name="T3" library="kumen" package="TO220" value="BTA16" x="38.1" y="39.37" rot="R90"/>
 <element name="R11" library="resistor" package="0207/10" value="330" x="27.94" y="39.37" rot="R225"/>
-<element name="R12" library="resistor" package="0207/10" value="180" x="78.105" y="36.83" rot="R180"/>
+<element name="R12" library="resistor" package="0207/10" value="220" x="78.105" y="36.83" rot="R180"/>
 <element name="CON2" library="#PaJa_konektory" package="WAGO256" value="WAGO256" x="15.24" y="24.13"/>
 <element name="CON3" library="#PaJa_konektory" package="WAGO256" value="WAGO256" x="15.24" y="43.18"/>
