File: PCB/ROwen_main.brd (EAGLE design)
At the start: 77.5 x 65.1 mm, 107 parts, among them CON1 MLW06_90°, CON2 MLW14_90°, CON3 S1G4_JUMP, CON4 S1G4_JUMP, CON5 MINI-USB-UX60-MB-5ST, CON6 S1G6_JUMP, IC1 STM32F042C, Q1 N-HEXFET-2D_SOT232-IRLL014N, SW1 P-B1720, SW2 P-B1720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

Commit message: small PCB updates
Parts:
- moved C4 2.93 mm to (37.9, 33.8)
- moved R16 2.93 mm to (36.4, 33.8)
- moved C11 2.93 mm to (39.5, 33.8)
- moved R17 2.93 mm to (34.8, 33.8)
- moved R_BOOT 2.93 mm to (33.2, 33.8)
- moved H4 1.00 mm to (73.0, 4.76)
- moved H3 0.71 mm to (4.45, 61.0)
- moved GND 0.32 mm to (4.45, 4.76)
- moved D4 0.32 mm to (75.6, 11.4)
- flipped C15 to the top, turned to 0 degrees
Connections:
- net N$34 renamed UART_RX
- net N$35 renamed UART_TX
Routing:
- net USB_DP: track 28.7 -> 37.5 mm
- net USB_DM: track 29.1 -> 37.7 mm
- net GND: track 513.9 -> 522.4 mm, vias 24 -> 25
- net +3V3: track 418.6 -> 423.7 mm, vias 10 -> 13
- net BOOT: track 9.25 -> 12.7 mm
- net V+: track 127.8 -> 130.8 mm, vias 3 -> 5
- net I2C_SDA: track 135.6 -> 138.1 mm
- net I2C_SCL: track 133.4 -> 135.3 mm

Commit message: Polygon improvement
Parts:
- removed GND: MOUNT-HOLE3.0, holes:3,0
- added H1: MOUNT-HOLE3.6, holes:3,6
- moved CON4 7.32 mm to (40.0, 9.37), turned to 0 degrees
- moved C10 0.16 mm to (41.1, 33.7)
- moved C11 0.16 mm to (39.5, 33.7)
- moved C4 0.16 mm to (37.9, 33.7)
- moved C6 0.16 mm to (47.5, 33.7)
- moved C7 0.16 mm to (49.1, 33.7)
- moved C9 0.16 mm to (45.9, 33.7)
- moved R16 0.16 mm to (36.4, 33.7)
- moved R17 0.16 mm to (34.8, 33.7)
- moved R53 0.16 mm to (42.7, 33.7)
- moved R54 0.16 mm to (44.3, 33.7)
- moved R_BOOT 0.16 mm to (33.2, 33.7)
- moved X1 0.16 mm to (43.5, 36.2)
Routing:
- net GND: track 522.4 -> 378.8 mm, vias 25 -> 60
- net +3V3: track 423.7 -> 430.3 mm, vias 13 -> 11
- net UART_TX: track 21.3 -> 16.1 mm
- net UART_RX: track 22.1 -> 18.1 mm
- net V+: track 130.8 -> 133.7 mm, vias 5 -> 7
Other:
- board size 77.5 x 65.1 mm -> 77.8 x 65.1 mm
- board text added: "2015"
- board text added: "ROwen"

Commit message: Manufactured version
Parts:
- flipped H1 to the bottom
Changed lines of the file:
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@@
 <layer number="45" name="Holes" color="7" fill="1" visible="no" active="yes"/>
 <layer number="46" name="Milling" color="3" fill="1" visible="no" active="yes"/>
-<layer number="47" name="Measures" color="7" fill="1" visible="no" active="yes"/>
+<layer number="47" name="Measures" color="7" fill="1" visible="yes" active="yes"/>
 <layer number="48" name="Document" color="7" fill="1" visible="no" active="yes"/>
 <layer number="49" name="Reference" color="7" fill="1" visible="no" active="yes"/>
@@
 <dimension x1="0.3175" y1="0.635" x2="76.8225" y2="0.635" x3="38.57" y3="-10.795" textsize="1.778" layer="248"/>
 <dimension x1="76.8225" y1="0.3175" x2="76.8225" y2="64.4425" x3="89.852503125" y3="32.38" textsize="1.778" layer="248"/>
-<dimension x1="0" y1="0.3175" x2="77.4575" y2="0.3175" x3="38.72875" y3="-3.4925" textsize="1.778" layer="47"/>
-<dimension x1="0" y1="65.395" x2="0" y2="0.3175" x3="-2.54" y3="32.85625" textsize="1.778" layer="47"/>
 <text x="21.9075" y="22.86" size="2.1844" layer="1" font="vector" ratio="15">ROwen</text>
 <text x="50.165" y="33.9725" size="2.1844" layer="1" font="vector" ratio="10">2015</text>
@@
 <element name="IOE1" library="kumen" package="SO24" value="PCA9555D" x="6.6675" y="47.625" rot="MR90"/>
 <element name="IOE2" library="kumen" package="SO24" value="PCA9555D" x="56.1975" y="47.625" rot="MR90"/>
-<element name="H1" library="holes" package="3,6" value="MOUNT-HOLE3.6" x="4.445" y="4.7625"/>
+<element name="H1" library="holes" package="3,6" value="MOUNT-HOLE3.6" x="4.445" y="4.7625" rot="MR0"/>
 </elements>
 <signals>
