File: PCB/ROwen_thermocouple.brd (EAGLE design)
At the start: 17.4 x 40.6 mm, 7 parts, among them CON1 MLW06_90°, K1 ARK550/2, K2 ARK550/2, K3 ARK550/2, K4 ARK550/2

Commit message: Manufactured version
Parts:
- CON1: device #PaJa_konektory:MLW06A -> !kumen:MLW06A
Changed lines of the file:
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@@
 </element>
 <element name="TEMP" library="kumen" package="SO8" value="TCN75A" x="11.43" y="30.48" rot="MR0"/>
-<element name="CON1" library="#PaJa_konektory" package="MLW06A" value="MLW06_90°" x="8.89" y="9.525" rot="R270"/>
+<element name="CON1" library="!kumen" package="MLW06A" value="MLW06_90°" x="8.89" y="9.525" rot="R270"/>
 </elements>
 <signals>
