File: PCB/ROwen_thermocouple.sch (EAGLE design)
At the start: 7 parts, among them CON1 MLW06_90°, K1 ARK550/2, K2 ARK550/2, K3 ARK550/2, K4 ARK550/2

Commit message: Manufactured version
Parts:
- CON1: device #PaJa_konektory:MLW06_90° -> !kumen:MLW06_90°
Changed lines of the file:
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@@
 <part name="GND5" library="supply1" deviceset="GND" device=""/>
 <part name="+3V3" library="supply1" deviceset="+3V3" device=""/>
-<part name="CON1" library="#PaJa_konektory" deviceset="MLW06" device="_90°"/>
+<part name="CON1" library="!kumen" deviceset="MLW06" device="_90°"/>
 <part name="GND1" library="supply1" deviceset="GND" device=""/>
 <part name="GND6" library="supply1" deviceset="GND" device=""/>
